Commit message: AY-04 unify temporary workcell station config and visual targets

File: src/carrier_description/urdf/machine_tending_cell.xacro (robot description, xacro)
@@ -5,5 +5,5 @@
     poses are not measured cell geometry or manufacturing CAD.
   -->
-  <xacro:macro name="machine_tending_cell" params="parent_link:=world">
+  <xacro:macro name="machine_tending_cell" params="parent_link:=world s1_xyz s1_rpy s1_size s2_xyz s2_rpy s2_size s3_xyz s3_rpy s3_size s4_xyz s4_rpy s4_size s5_xyz s5_rpy s5_size">
     <link name="cell_floor">
       <visual>
@@ -17,37 +17,37 @@
     </joint>
     <link name="station_s1_raw">
-      <visual><origin xyz="0 0 0.35"/><geometry><box size="0.45 0.45 0.70"/></geometry>
+      <visual><origin xyz="0 0 ${float(s1_size.split()[2]) / 2.0}"/><geometry><box size="${s1_size}"/></geometry>
         <material name="station_raw_material"><color rgba="0.20 0.45 0.85 1"/></material></visual>
     </link>
     <joint name="world_to_station_s1_raw" type="fixed">
-      <parent link="${parent_link}"/><child link="station_s1_raw"/><origin xyz="0.75 0.85 0"/>
+      <parent link="${parent_link}"/><child link="station_s1_raw"/><origin xyz="${s1_xyz}" rpy="${s1_rpy}"/>
     </joint>
     <link name="station_s2_staging">
-      <visual><origin xyz="0 0 0.35"/><geometry><box size="0.45 0.45 0.70"/></geometry>
+      <visual><origin xyz="0 0 ${float(s2_size.split()[2]) / 2.0}"/><geometry><box size="${s2_size}"/></geometry>
         <material name="station_staging_material"><color rgba="0.90 0.70 0.12 1"/></material></visual>
     </link>
     <joint name="world_to_station_s2_staging" type="fixed">
-      <parent link="${parent_link}"/><child link="station_s2_staging"/><origin xyz="0.15 1.05 0"/>
+      <parent link="${parent_link}"/><child link="station_s2_staging"/><origin xyz="${s2_xyz}" rpy="${s2_rpy}"/>
     </joint>
     <link name="station_s3_machine">
-      <visual><origin xyz="0 0 0.60"/><geometry><box size="0.75 0.70 1.20"/></geometry>
+      <visual><origin xyz="0 0 ${float(s3_size.split()[2]) / 2.0}"/><geometry><box size="${s3_size}"/></geometry>
         <material name="station_machine_material"><color rgba="0.25 0.28 0.32 1"/></material></visual>
     </link>
     <joint name="world_to_station_s3_machine" type="fixed">
-      <parent link="${parent_link}"/><child link="station_s3_machine"/><origin xyz="-0.65 0.75 0"/>
+      <parent link="${parent_link}"/><child link="station_s3_machine"/><origin xyz="${s3_xyz}" rpy="${s3_rpy}"/>
     </joint>
     <link name="station_s4_output">
-      <visual><origin xyz="0 0 0.35"/><geometry><box size="0.45 0.45 0.70"/></geometry>
+      <visual><origin xyz="0 0 ${float(s4_size.split()[2]) / 2.0}"/><geometry><box size="${s4_size}"/></geometry>
         <material name="station_output_material"><color rgba="0.85 0.42 0.12 1"/></material></visual>
     </link>
     <joint name="world_to_station_s4_output" type="fixed">
-      <parent link="${parent_link}"/><child link="station_s4_output"/><origin xyz="-0.75 -0.45 0"/>
+      <parent link="${parent_link}"/><child link="station_s4_output"/><origin xyz="${s4_xyz}" rpy="${s4_rpy}"/>
     </joint>
     <link name="station_s5_finished">
-      <visual><origin xyz="0 0 0.35"/><geometry><box size="0.45 0.45 0.70"/></geometry>
+      <visual><origin xyz="0 0 ${float(s5_size.split()[2]) / 2.0}"/><geometry><box size="${s5_size}"/></geometry>
         <material name="station_finished_material"><color rgba="0.18 0.70 0.35 1"/></material></visual>
     </link>
     <joint name="world_to_station_s5_finished" type="fixed">
-      <parent link="${parent_link}"/><child link="station_s5_finished"/><origin xyz="0.35 -0.95 0"/>
+      <parent link="${parent_link}"/><child link="station_s5_finished"/><origin xyz="${s5_xyz}" rpy="${s5_rpy}"/>
     </joint>
     <!-- Three joints make visual workpiece state changes observable in /joint_states. -->

File: src/carrier_description/urdf/ur5_with_test_tool.xacro (robot description, xacro)
@@ -21,4 +21,21 @@
   <xacro:arg name="tf_prefix" default=""/>
   <xacro:arg name="include_workcell" default="true"/>
+  <!-- Standalone Xacro fallback values mirror machine_tending.json. Both ROS
+       launch entry points override them from the installed plan at runtime. -->
+  <xacro:arg name="station_s1_xyz" default="0.75 0.85 0"/>
+  <xacro:arg name="station_s1_rpy" default="0 0 0"/>
+  <xacro:arg name="station_s1_size" default="0.45 0.45 0.70"/>
+  <xacro:arg name="station_s2_xyz" default="0.15 1.05 0"/>
+  <xacro:arg name="station_s2_rpy" default="0 0 0"/>
+  <xacro:arg name="station_s2_size" default="0.45 0.45 0.70"/>
+  <xacro:arg name="station_s3_xyz" default="-0.65 0.75 0"/>
+  <xacro:arg name="station_s3_rpy" default="0 0 0"/>
+  <xacro:arg name="station_s3_size" default="0.75 0.70 1.20"/>
+  <xacro:arg name="station_s4_xyz" default="-0.75 -0.45 0"/>
+  <xacro:arg name="station_s4_rpy" default="0 0 0"/>
+  <xacro:arg name="station_s4_size" default="0.45 0.45 0.70"/>
+  <xacro:arg name="station_s5_xyz" default="0.35 -0.95 0"/>
+  <xacro:arg name="station_s5_rpy" default="0 0 0"/>
+  <xacro:arg name="station_s5_size" default="0.45 0.45 0.70"/>
   <!-- World -->
   <link name="world"/>
@@ -27,5 +44,10 @@
     <xacro:include
       filename="$(find carrier_description)/urdf/machine_tending_cell.xacro"/>
-    <xacro:machine_tending_cell parent_link="world"/>
+    <xacro:machine_tending_cell parent_link="world"
+      s1_xyz="$(arg station_s1_xyz)" s1_rpy="$(arg station_s1_rpy)" s1_size="$(arg station_s1_size)"
+      s2_xyz="$(arg station_s2_xyz)" s2_rpy="$(arg station_s2_rpy)" s2_size="$(arg station_s2_size)"
+      s3_xyz="$(arg station_s3_xyz)" s3_rpy="$(arg station_s3_rpy)" s3_size="$(arg station_s3_size)"
+      s4_xyz="$(arg station_s4_xyz)" s4_rpy="$(arg station_s4_rpy)" s4_size="$(arg station_s4_size)"
+      s5_xyz="$(arg station_s5_xyz)" s5_rpy="$(arg station_s5_rpy)" s5_size="$(arg station_s5_size)"/>
   </xacro:if>
   <!-- UR5 -->
